File: Main/Main.kicad_pcb (KiCad board)
At the start: 2 copper layers, 100 x 66 mm, 117 parts, among them IC1 Seed_XIAO_ESP32C3, J1 PWR_IN, J11 Conn_01x05, J2 Ball, J3 MotorDriver, J4 Line, J5 Camera, J6 Speaker, J7 Catch, J8 ST-LINK, J9 USB_C_Receptacle_USB2.0_16P, Q1 MMBT3904, SW2 SW_Push, SW3 SW_Push, SW4 SW_Push, SW5 SW_Push, SW6 SW_Push, U1 STM32F446RETx, U2 AZ1117CH-3_3TRG1, U3 STM32F103CBTx, Y1 8MHz, Y2 8mHz

Commit message: Ver-1.2
Parts:
- moved G*** 0.25 mm to (163.5, 84.0)
Changed lines of the file:
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@@
 	(footprint "Logo:JLCPCB"
 		(layer "F.Cu")
-		(at 163.25 84)
+		(at 163.5 84)
 		(property "Reference" "G***"
 			(at 0 0 0)
@@
 	)
 	(gr_line
-		(start 173.75 81.5)
-		(end 173.75 66.5)
-		(stroke
-			(width 0.15)
-			(type default)
-		)
-		(layer "F.SilkS")
-	)
-	(gr_line
 		(start 143.75 130.25)
 		(end 143.75 113.75)
@@
 	)
 	(gr_line
-		(start 130.25 66.25)
-		(end 130.25 81.5)
-		(stroke
-			(width 0.15)
-			(type default)
-		)
-		(layer "F.SilkS")
-	)
-	(gr_line
 		(start 193.5 68.5)
 		(end 207.75 68.5)
@@
 	)
 	(gr_line
-		(start 154 81.5)
-		(end 157.5 81.5)
-		(stroke
-			(width 0.15)
-			(type default)
-		)
-		(layer "F.SilkS")
-	)
-	(gr_line
 		(start 133.5 130.25)
 		(end 143.75 130.25)
@@
 	)
 	(gr_line
-		(start 158.25 81.5)
-		(end 173.75 81.5)
-		(stroke
-			(width 0.15)
-			(type default)
-		)
-		(layer "F.SilkS")
-	)
-	(gr_line
 		(start 192 71.5)
 		(end 192 70.75)
@@
 	)
 	(gr_line
-		(start 130.25 81.5)
-		(end 135.5 81.5)
-		(stroke
-			(width 0.15)
-			(type default)
-		)
-		(layer "F.SilkS")
-	)
-	(gr_line
 		(start 130.75 110.25)
 		(end 140.5 110.25)
@@
 		(stroke
 			(width 0.15)
-			(type default)
-		)
-		(layer "F.SilkS")
-	)
-	(gr_line
-		(start 136.25 81.5)
-		(end 151 81.5)
-		(stroke
-			(width 0.15)
-			(type default)
-		)
-		(layer "F.SilkS")
-	)
-	(gr_line
-		(start 151 81.5)
-		(end 154 81.5)
-		(stroke
-			(width 0.15)
